File: eagle/clk_master.brd (EAGLE design)
At the start: 76.2 x 50.8 mm, 69 parts, among them U1 74LVCU04A, U2 MCP1824ST-3302E, U3 ATXMEGA16A4U, U4 ENC28J60, U5 TESEO-LIV3R, U8 74LVC74A, U9 74LVC86A

Commit message: specifiy VCTCXO part number
Parts:
- U6: value (none) -> SIT5156AI-FD-33VT-25.000000Y
Changed lines of the file:
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@@
 <attribute name="NAME" x="33.655" y="17.145" size="1.27" layer="25" rot="R90"/>
 </element>
-<element name="U6" library="crystal" library_urn="urn:adsk.eagle:library:204" package="ASF" package3d_urn="urn:adsk.eagle:package:12096/1" value="" x="34.925" y="13.335" smashed="yes" rot="R270">
+<element name="U6" library="crystal" library_urn="urn:adsk.eagle:library:204" package="ASF" package3d_urn="urn:adsk.eagle:package:12096/1" value="SIT5156AI-FD-33VT-25.000000Y" x="34.925" y="13.335" smashed="yes" rot="R270">
 <attribute name="NAME" x="36.54" y="17.55" size="1.27" layer="25" rot="R180"/>
 <attribute name="VALUE" x="32.175" y="15.585" size="1.27" layer="27" rot="R270"/>
